Commit message: modified:   wheeled_robin/package.xml 	modified:   wheeled_robin_bringup/launch/includes/mobile_base.launch.xml 	modified:   wheeled_robin_bringup/launch/includes/mobile_base_fake.launch.xml 	modified:   wheeled_robin_bringup/launch/includes/robot.launch.xml 	modified:   wheeled_robin_description/urdf/wheeled_robin.urdf.xacro 	deleted:    wheeled_robin_driver/src/wheeled_robin_driver.py 	modified:   wheeled_robin_driver/src/wheeled_robin_driver/wheeled_robin_driver.py 	modified:   wheeled_robin_driver/src/wheeled_robin_driver/wheeled_robin_driver.pyc 	modified:   wheeled_robin_node/msg/WheeledRobinSensorState.msg 	modified:   wheeled_robin_node/nodes/test_driver.py 	modified:   wheeled_robin_node/nodes/wheeled_node.py 	modified:   wheeled_robin_node/src/wheeled_robin_node/wheeled_robin_sensor_handler.py 	modified:   wheeled_robin_node/src/wheeled_robin_node/wheeled_robin_sensor_handler.pyc 	wheeled_robin_bringup/apps/ 	wheeled_robin_bringup/concert/ 	wheeled_robin_bringup/icons/ 	wheeled_robin_bringup/launch/minimal_fake_with_appmanager.launch 	wheeled_robin_bringup/launch/minimal_with_appmanager.launch 	wheeled_robin_bringup/launch/paired_public.launch

File: wheeled_robin_description/urdf/wheeled_robin.urdf.xacro (robot description, xacro)
@@ -9,20 +9,4 @@
 	      <color rgba="0.0 0.8 0.0 1.0"/>
 	  </material>
-	  <!-- base_footprint is a fictitious link(frame) that is on the ground right below base_link origin, navigation stack depends on this frame -->
-	  <link name="base_footprint">
-	    <!--<visual>
-	      <origin xyz="0 0 0" rpy="0 0 0" />
-	      <geometry>
-	        <box size="0.001 0.001 0.001" />
-	      </geometry>
-	      <material name="Green" />
-	    </visual>
-	    <collision>
-	      <origin xyz="0 0 0.017" rpy="0 0 0" />
-	      <geometry>
-	       <box size="0.001 0.001 0.001" />
-	      </geometry>
-	    </collision>-->
-	  </link>
 	  <link name="base_link">
 	    <!--<inertial>
@@ -45,9 +29,4 @@
 	    </collision>-->
 	  </link>
-	  <joint name="base_footprint_joint" type="fixed">
-	    <origin xyz="0 0 0.055" rpy="0 0 0" />
-	    <parent link="base_footprint"/>
-	    <child link="base_link" />
-	  </joint>
 	  <link name="left_wheel_link">
 	    <!--<inertial>
@@ -87,6 +66,6 @@
 	      <origin xyz="0 0 0" rpy="0 1.5707 1.5707" />
 	      <geometry>
-	        <mesh filename="package://wheeled_robin_description/meshes/reifenascii.stl"/>-->
-	        <!--<cylinder radius="0.055" length = "0.05"/>-->
+	        <!--<mesh filename="package://wheeled_robin_description/meshes/reifenascii.stl"/>-->
+	        <cylinder radius="0.055" length = "0.05"/>
 	      </geometry>
 	      <material name="Green" />

Commit message: modified:   wheeled_robin_bringup/launch/3dsensor.launch 	modified:   wheeled_robin_bringup/launch/includes/mobile_base.launch.xml 	modified:   wheeled_robin_bringup/launch/includes/mobile_base_fake.launch.xml 	modified:   wheeled_robin_description/urdf/wheeled_robin.urdf.xacro 	modified:   wheeled_robin_description/urdf/wheeled_robin_library.urdf.xacro

File: wheeled_robin_description/urdf/wheeled_robin.urdf.xacro (robot description, xacro)
@@ -97,5 +97,25 @@
 	    <child link="gyro_link"/>
 	  </joint>-->
-	  <link name="laser">
+	  <link name="camera_link">
+	    <!--<visual>
+	      <geometry>
+	        <box size="0 0 0.5" />
+	      </geometry>
+	      <material name="Green" />
+	    </visual>
+	    <inertial>
+	      <mass value="0.001" />
+	      <origin xyz="0 0 0" />
+	      <inertia ixx="0.0001" ixy="0.0" ixz="0.0"
+	        iyy="0.0001" iyz="0.0"
+	        izz="0.0001" />
+	    </inertial>-->
+	  </link>
+	  <joint name="camera_joint" type="fixed">
+	    <origin xyz="0.1 0.0315 0.5" rpy="0 0 0" />
+	    <parent link="base_link" />
+	    <child link="camera_link" />
+	  </joint>
+	  <link name="laser_link">
 	    <!--<visual>
 	      <geometry>
@@ -115,5 +135,5 @@
 	    <origin xyz="-0.065 0 0.075" rpy="0 0 0" />
 	    <parent link="base_link" />
-	    <child link="laser" />
+	    <child link="laser_link" />
 	  </joint>
 	  <!-- Simulation sensors -->

File: wheeled_robin_description/urdf/wheeled_robin_library.urdf.xacro (robot description, xacro)
@@ -6,5 +6,5 @@
   <!-- General -->
   <xacro:include filename="$(find turtlebot_description)/urdf/common_properties.urdf.xacro"/>
-  <xacro:include filename="$(find wheeled_robin_description)/urdf/wheeled_robin_properties.urdf.xacro"/>
+  <!--<xacro:include filename="$(find wheeled_robin_description)/urdf/wheeled_robin_properties.urdf.xacro"/>-->
   <!-- Bases -->
   <xacro:include filename="$(find wheeled_robin_description)/urdf/wheeled_robin.urdf.xacro"/>

Commit message: modified:   urdf/wheeled_robin.urdf.xacro

File: wheeled_robin_description/urdf/wheeled_robin.urdf.xacro (robot description, xacro)
@@ -6,6 +6,6 @@
   <property name="base_y" value="0.33" />
 	<xacro:macro name="wheeled_robin">
-	  <material name="Green">
-	      <color rgba="0.0 0.8 0.0 1.0"/>
+	  <material name="Grey">
+	      <color rgba="0.7 0.7 0.7 1.0"/>
 	  </material>
 	  <link name="base_link">
@@ -17,8 +17,10 @@
 	    </inertial> -->
 	    <visual>
-	      <origin xyz=" 0 0 0.07" rpy="0 0 0" />
-	      <geometry>
-	        <box size="0.124 0.19 0.2" />
-	      </geometry>
+	      <!-- <origin xyz=" 0 0 0.07" rpy="0 0 0" /> -->
+		<origin xyz=" 0 0 0" rpy="-1.5707 0 0" />
+	      <geometry>
+		<mesh filename="package://wheeled_robin_description/meshes/segway.stl"/>
+	      </geometry>
+		<material name="Grey" />
 	    </visual>
 	    <!--<collision>
@@ -37,9 +39,9 @@
 	    </inertial> -->
 	    <visual>
-	      <origin xyz="0 0 0" rpy="0 1.5707 1.5707" />
-	      <geometry>
-	        <cylinder radius="0.055" length = "0.05"/>
-	      </geometry>
-	      <material name="Green" />
+	      <origin xyz="0 0 0" rpy="-1.5707 0 0" />
+	      <geometry>
+		<mesh filename="package://wheeled_robin_description/meshes/wheel.stl"/>
+	      </geometry>
+		<material name="Grey" />
 	    </visual>
 	    <!--<collision>
@@ -51,5 +53,6 @@
 	  </link>
 	  <joint name="left_wheel_joint" type="continuous">
-	    <origin xyz="0 0.118 0" rpy="0 0 0"/>
+	    <!-- <origin xyz="0 0.118 0" rpy="0 0 0"/> -->
+		<origin xyz="0 0.0925 0" rpy="0 0 0"/>
 	    <parent link="base_link"/>
 	    <child link="left_wheel_link"/>
@@ -64,10 +67,9 @@
 	    </inertial> -->
 	    <visual>
-	      <origin xyz="0 0 0" rpy="0 1.5707 1.5707" />
-	      <geometry>
-	        <!--<mesh filename="package://wheeled_robin_description/meshes/reifenascii.stl"/>-->
-	        <cylinder radius="0.055" length = "0.05"/>
-	      </geometry>
-	      <material name="Green" />
+	      <origin xyz="0 0 0" rpy=" 1.5707 0 0" />
+	      <geometry>
+		<mesh filename="package://wheeled_robin_description/meshes/wheel.stl"/>
+	      </geometry>
+	      <material name="Grey" />
 	    </visual>
 	    <!--<collision>
@@ -79,5 +81,5 @@
 	  </link>
 	  <joint name="right_wheel_joint" type="continuous">
-	    <origin xyz="0 -0.118 0" rpy="0 0 0"/>
+	    <origin xyz="0 -0.0925 0" rpy="0 0 0"/>
 	    <parent link="base_link"/>
 	    <child link="right_wheel_link"/>
@@ -97,5 +99,17 @@
 	    <child link="gyro_link"/>
 	  </joint>-->
-	  <link name="camera_link">
+	    <!--<inertial>
+	      <mass value="0.001" />
+	      <origin xyz="0 0 0" />
+	      <inertia ixx="0.0001" ixy="0.0" ixz="0.0"
+	        iyy="0.0001" iyz="0.0"
+	        izz="0.0001" />
+	    </inertial>-->
+	  <joint name="camera_joint" type="fixed">
+	    <origin xyz="0.045 0 0.54" rpy="0 0 0" />
+	    <parent link="base_link" />
+	    <child link="camera_link" />
+	  </joint>
+	  <link name="laser_link">
 	    <!--<visual>
 	      <geometry>
@@ -112,34 +126,90 @@
 	    </inertial>-->
 	  </link>
-	  <joint name="camera_joint" type="fixed">
-	    <origin xyz="0.1 0.0315 0.5" rpy="0 0 0" />
-	    <parent link="base_link" />
-	    <child link="camera_link" />
-	  </joint>
-	  <link name="laser_link">
-	    <!--<visual>
-	      <geometry>
-	        <box size="0 0 0.5" />
-	      </geometry>
-	      <material name="Green" />
-	    </visual>
-	    <inertial>
-	      <mass value="0.001" />
-	      <origin xyz="0 0 0" />
-	      <inertia ixx="0.0001" ixy="0.0" ixz="0.0"
-	        iyy="0.0001" iyz="0.0"
-	        izz="0.0001" />
-	    </inertial>-->
-	  </link>
 	  <joint name="laser_joint" type="fixed">
-	    <origin xyz="-0.065 0 0.075" rpy="0 0 0" />
-	    <parent link="base_link" />
+	    <origin xyz="0.031 0 0.016" rpy="0 0 0" />
+	    <parent link="camera_link" />
 	    <child link="laser_link" />
 	  </joint>
-	  <!-- Simulation sensors -->
-	  <!--<sim_wheeled_robin/>
-	  <sim_wheeled_robin_wall_sensor/>
-	  <sim_wheeled_robin_cliff_sensors/>
-	  <sim_imu/>-->
+<!-- ####### Kinect Frames ######## -->
+      <link name="camera_link">
+    <!-- 	<visual>
+     	<origin xyz="0 0 0" rpy="0 0 ${M_PI/2}"/>
+     <geometry>
+       <mesh filename="package://turtlebot_description/meshes/sensors/kinect.dae"/>
+      </geometry>
+    </visual>
+	  <collision>
+      <origin xyz="0.0 0.0 0.0" rpy="0 0 0"/>
+	    <geometry>
+	      <box size="0.07271 0.27794 0.073"/>
+	    </geometry>
+	  </collision> -->
+    <inertial>
+      <mass value="0.001" />
+      <origin xyz="0 0 0" />
+      <inertia ixx="0.0001" ixy="0.0" ixz="0.0"
+               iyy="0.0001" iyz="0.0"
+               izz="0.0001" />
+    </inertial>
+  </link>
+    <joint name="camera_rgb_joint" type="fixed">
+      <origin xyz="0.031 -0.0125 0.016" rpy="0 0 0"/>
+      <parent link="camera_link"/>
+      <child link="camera_rgb_frame" />
+    </joint>
+    <link name="camera_rgb_frame">
+      <inertial>
+        <mass value="0.001" />
+        <origin xyz="0 0 0" />
+        <inertia ixx="0.0001" ixy="0.0" ixz="0.0"
+                 iyy="0.0001" iyz="0.0"
+                 izz="0.0001" />
+      </inertial>
+    </link>
+    <joint name="camera_rgb_optical_joint" type="fixed">
+      <origin xyz="0 0 0" rpy="${-M_PI/2} 0 ${-M_PI/2}" />
+      <parent link="camera_rgb_frame" />
+      <child link="camera_rgb_optical_frame" />
+    </joint>
+    <link name="camera_rgb_optical_frame">
+      <inertial>
+        <mass value="0.001" />
+        <origin xyz="0 0 0" />
+        <inertia ixx="0.0001" ixy="0.0" ixz="0.0"
+                 iyy="0.0001" iyz="0.0"
+                 izz="0.0001" />
+      </inertial>
+    </link>
+  <!-- The fixed joints & links below are usually published by static_transformers launched by the OpenNi launch
+       files. However, for Gazebo simulation we need them, so we add them here.
+       (Hence, don't publish them additionally!) -->
+	<joint name="camera_depth_joint" type="fixed">
+	  <origin xyz="0 0.025 0" rpy="0 0 0" />
+	  <parent link="camera_rgb_frame" />
+	  <child link="camera_depth_frame" />
+	</joint>
+	<link name="camera_depth_frame">
+    <inertial>
+      <mass value="0.001" />
+      <origin xyz="0 0 0" />
+      <inertia ixx="0.0001" ixy="0.0" ixz="0.0"
+               iyy="0.0001" iyz="0.0"
+               izz="0.0001" />
+    </inertial>
+	</link>
+	<joint name="camera_depth_optical_joint" type="fixed">
+	  <origin xyz="0 0 0" rpy="${-M_PI/2} 0 ${-M_PI/2}" />
+	  <parent link="camera_depth_frame" />
+	  <child link="camera_depth_optical_frame" />
+	</joint>
+	<link name="camera_depth_optical_frame">
+    <inertial>
+      <mass value="0.001" />
+      <origin xyz="0 0 0" />
+      <inertia ixx="0.0001" ixy="0.0" ixz="0.0"
+               iyy="0.0001" iyz="0.0"
+               izz="0.0001" />
+    </inertial>
+	</link>
 	</xacro:macro>
 </robot>
